File: hardware/OPNhydro_r1/OPNhydro_r1.kicad_sch (KiCad schematic)
At the start: 82 parts, among them J1 JACK_5MM, J10 BNC_EC, J11 Float_Low, J12 BME280, J13 BNC_DO, J14 Float_High, J17 Main_Pump, J18 pH_Up_Pump, J19 pH_Down_Pump, J2 EZO-pH, J20 Nutrient_A, J21 Nutrient_B, J22 ATO_Valve, J3 BH1750, J4 1-Wire, J5 EZO-EC, J6 OLED, J7 HC-SR04, J8 EZO-DO, J9 BNC_pH, Q2 IRLZ44N, Q3 IRLZ44N, Q4 IRLZ44N, Q5 IRLZ44N, Q6 IRLZ44N, Q7 IRLZ44N, U1 SI2301, U2 TPS62933

Commit message: update design and schematic
Parts:
- removed C1: 100nF, Capacitor_SMD:C_0805_2012Metric, symbol Device:C
- removed J10: BNC_EC, Connector:BNC_TEConnectivity_1478204_Vertical, symbol Connector:Conn_01x02_Pin
- removed J13: BNC_DO, Connector:BNC_TEConnectivity_1478204_Vertical, symbol Connector:Conn_01x02_Pin
- removed J2: EZO-pH, Connector_JST:JST_PH_B4B-PH-K_1x04_P2.00mm_Vertical, symbol Connector:Conn_01x04_Pin
- removed J5: EZO-EC, Connector_JST:JST_PH_B4B-PH-K_1x04_P2.00mm_Vertical, symbol Connector:Conn_01x04_Pin
- removed J8: EZO-DO, Connector_JST:JST_PH_B4B-PH-K_1x04_P2.00mm_Vertical, symbol Connector:Conn_01x04_Pin
- removed J9: BNC_pH, Connector:BNC_TEConnectivity_1478204_Vertical, symbol Connector:Conn_01x02_Pin
- removed R1, R3: 4.7k, Resistor_SMD:R_0805_2012Metric, symbol Device:R
- added C12, C13, C16, C21: 100nF, Coert-Vonk:CAP X7R 100nF ±10 25V 0805, symbol Coert-Vonk:CAP X7R 100nF ±10% 25V 0805
- added C14, C17: 10μF, Coert-Vonk:CAP X7R 10μF ±10 16V 0805, symbol Coert-Vonk:CAP X7R 10μF ±10% 16V 0805
- added C18, C22: 10nF, Coert-Vonk:CAP X7R 10nF ±10% 50V 0805, symbol Coert-Vonk:CAP X7R 10nF ±10% 50V 0805
- added EZO: PH, symbol Coert-Vonk:EVAL EZO pH
- added FB7, FB8: 330Ω at 100MHz, Coert-Vonk:FERRITE BEAD 330Ω 0805, symbol Coert-Vonk:FERRITE BEAD 330Ω 0805
- added J15: PH, Coert-Vonk:CONN BNC JACK RA 50Ω, symbol Coert-Vonk:CONN BNC JACK RA 50Ω 5227161-6
- added R25, R26: 4k7, Coert-Vonk:RES 4.7kΩ 0805, symbol Coert-Vonk:RES 4.7kΩ ±5% 1/4W 0805
- added R27: 16k9, Coert-Vonk:RES 16.9kΩ ±1 18W 0805, symbol Coert-Vonk:RES 16.9kΩ ±1% 1/8W 0805
- added R28: 10k, Coert-Vonk:RES 10kΩ 0805, symbol Coert-Vonk:RES 10kΩ ±1% 1/8W 0805
- added U3: ADM3260, Coert-Vonk:IC ISOLTR 2.5KV 2CH I2C 20SSOP ADM3260, symbol Coert-Vonk:IC ISOLTR 2.5KV 2CH I2C 20SSOP ADM3260
Connections:
- net BOOT is gone; now on net FLOAT_LOW: PCB1.J1_7 (IO0/ADC0)
- net +12V: no longer C4.2, C5.2, U1.3 (D), U2.3 (VIN)
- net +3V3: now also J4.1 (Pin_1)
- net +5V: no longer C10.2, C9.2, DC1.3 (VI), L1.2, PCB1.J1_14 (5V0), R23.2
- net ATO_VALVE: now also PCB1.J1_6 (IO7/SPI_MOSI)
- net FLOAT_HIGH: now also PCB1.J1_8 (IO1/ADC1)
- net GND: now also J4.3 (Pin_3), C12.1, C17.1, C21.1, C22.1, U3.1 (GND_{P}), U3.10 (GND_{P}), U3.5 (GND_{P}), U3.7 (GND_{P})
- net I2C_SCL: now also R25.1, U3.2 (SCL_{2})
- net I2C_SDA: now also R26.1, U3.3 (SDA_{2})
- net ONEWIRE: now also J4.2 (Pin_2)
- net ONE_WIRE: now also PCB1.J1_12 (IO2/SPI_MISO)
- net PUMP_MAIN: now also PCB1.J1_10 (IO10)
- net PUMP_NUT_A: now also PCB1.J3_9 (IO19)
- net PUMP_NUT_B: now also PCB1.J3_8 (IO20)
- net PUMP_PH_DN: now also PCB1.J3_4 (IO15)
- net PUMP_PH_UP: now also PCB1.J1_11 (IO11)
- net US_ECHO: now also PCB1.J1_13 (IO3/ADC3)
- net US_TRIG: now also PCB1.J3_11 (IO9/ADC9)
- net +3.3V renamed 3V3
- net 3V3: now also C12.2, C17.2, C21.2, C22.2, R25.2, R26.2, U3.4 (VDD_{P}), U3.9 (V_{IN})
- new net: R27.1, R28.2, U3.13 (VSEL)
- new net: C16.2, C18.2, EZO.6 (VCC), FB8.1, R27.2, U3.17 (VDD_{ISO})
- new net: C13.2, C14.2, FB8.2, U3.12 (V_{ISO})
- new net: C13.1, C14.1, C16.1, C18.1, FB7.2, R28.1, U3.11 (GND_{ISO}), U3.14 (GND_{ISO}), U3.16 (GND_{ISO}), U3.20 (GND_{ISO})
- new net: EZO.1 (GND), FB7.1
- new net: EZO.2 (TX/SCL), U3.19 (SCL_{1})
- new net: EZO.3 (RX/SDA), U3.18 (SDA_{1})
- new net: EZO.4 (PGND), J15.G (GND)
- new net: EZO.5 (PRB), J15.S
- new net 12V: C4.2, C5.2, U1.3 (D), U2.3 (VIN)
- new net 5V: C10.2, C9.2, DC1.3 (VI), L1.2, PCB1.J1_14 (5V0), R23.2
- new net EZO_PDIS: U3.8 (PDIS)
- no-connect marks 6 -> 9
Other:
- note added: "ANALOG→I2C"
- note added: "Dual function pin considerations: IO8 is used for RGB LED on the DevKitC => reserved. IO9 has internal ~45kΩ pullup. US_TRIG is a non-critical output, initialized after boot => OK. IO15 has a 10kΩ pulldown due to the MOSFET driver. This will disable ESP32 ROM boot messages. IO17 is driven by the CP2102N UART TX output => reserved. D+/D- are used for Serial Logging, Code Upload and JTAG debugging.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"
- note added: "ESP32-C6-DevKitC"
- note added: "I2C BUS"
- note added: "ISOLATOR"
- note added: "PH SENSOR"
- note removed: "BNC Probe Connectors"
- note removed: "ESP32-C6-DevKitC-1-N8 HEADERS"
- note removed: "I2C BUS & SENSOR CONNECTORS"
- note removed: "To EZO PRB"
- moved on the sheet: J12, J3, J4, J6, R2

Commit message: add pump ctrl and power buffers
Parts:
- removed C10: 10μF, Coert-Vonk:CAP CER 10µF 25V 0805, symbol Coert-Vonk:CAP CER 10µF 25V 0805
- removed C6: 100nF, Capacitor_SMD:C_0805_2012Metric, symbol Device:C
- removed D2: WS2812B, LED_SMD:LED_WS2812B_PLCC4_5.0x5.0mm_P3.2mm, symbol LED:WS2812B
- removed D3, D4, D5, D6, D7, D8: SS34, Diode_SMD:D_SMA_Handsoldering, symbol Device:D_Schottky
- removed J17: Main_Pump, Connector_Phoenix_MSTB:PhoenixContact_MSTBA_2,5_2-G-5,08_1x02_P5.08mm_Horizontal, symbol Connector:Conn_01x02_Pin
- removed J18: pH_Up_Pump, Connector_Phoenix_MSTB:PhoenixContact_MSTBA_2,5_2-G-5,08_1x02_P5.08mm_Horizontal, symbol Connector:Conn_01x02_Pin
- removed J19: pH_Down_Pump, Connector_Phoenix_MSTB:PhoenixContact_MSTBA_2,5_2-G-5,08_1x02_P5.08mm_Horizontal, symbol Connector:Conn_01x02_Pin
- removed J20: Nutrient_A, Connector_Phoenix_MSTB:PhoenixContact_MSTBA_2,5_2-G-5,08_1x02_P5.08mm_Horizontal, symbol Connector:Conn_01x02_Pin
- removed J21: Nutrient_B, Connector_Phoenix_MSTB:PhoenixContact_MSTBA_2,5_2-G-5,08_1x02_P5.08mm_Horizontal, symbol Connector:Conn_01x02_Pin
- removed J22: ATO_Valve, Connector_Phoenix_MSTB:PhoenixContact_MSTBA_2,5_2-G-5,08_1x02_P5.08mm_Horizontal, symbol Connector:Conn_01x02_Pin
- removed Q2, Q3, Q4, Q5, Q6, Q7: IRLZ44N, Package_TO_SOT_THT:TO-220-3_Vertical, symbol Device:Q_NMOS_GDS
- removed R10, R11, R12, R13, R14, R15, R16: 100R, Resistor_SMD:R_0805_2012Metric, symbol Device:R
- removed R17, R18, R19, R20, R21, R22: 10k, Resistor_SMD:R_0805_2012Metric, symbol Device:R
- added C1: 1000μF, Coert-Vonk:CAP ALUM POLY 1000μF ±20 6.3V, symbol Coert-Vonk:CAP ALUM POLY 1000μF ±20% 6.3V
- added C6: 2200μF, Coert-Vonk:CAP ALUM 2200μF ±20 25V RADIAL, symbol Coert-Vonk:CAP ALUM 2200μF ±20% 25V RADIAL
- added D3, D4, D5, D6, D7, D9: SS34, Coert-Vonk:DIODE SCHOTTKY 40V 3A DIOM7959X265N DO214AB, symbol Coert-Vonk:DIODE SCHOTTKY 40V 3A DIOM7959X265N DO214AB
- added HDR1: PUMP_MAIN, Coert-Vonk:TERM BLOCK HDR 2POS RA 3.81mm 1803277, symbol Coert-Vonk:TERM BLOCK HDR 2POS RA 3.81mm
- added HDR2: ATO_VALVE, Coert-Vonk:TERM BLOCK HDR 2POS RA 3.81mm 1803277, symbol Coert-Vonk:TERM BLOCK HDR 2POS RA 3.81mm
- added HDR3: PUMP_PH_UP, Coert-Vonk:TERM BLOCK HDR 2POS RA 3.81mm 1803277, symbol Coert-Vonk:TERM BLOCK HDR 2POS RA 3.81mm
- added HDR4: PUMP_PH_DN, Coert-Vonk:TERM BLOCK HDR 2POS RA 3.81mm 1803277, symbol Coert-Vonk:TERM BLOCK HDR 2POS RA 3.81mm
- added HDR5: PUMP_NUT_A, Coert-Vonk:TERM BLOCK HDR 2POS RA 3.81mm 1803277, symbol Coert-Vonk:TERM BLOCK HDR 2POS RA 3.81mm
- added HDR6: PUMP_NUT_B, Coert-Vonk:TERM BLOCK HDR 2POS RA 3.81mm 1803277, symbol Coert-Vonk:TERM BLOCK HDR 2POS RA 3.81mm
- added Q1: 2N7002K, Coert-Vonk:MOSFET N-CH 55V 42A IRLR2905TRPBF DPAK, symbol Coert-Vonk:MOSFET N-CH 55V 42A IRLR2905TRPBF DPAK
- added Q2, Q3, Q4, Q5, Q8: AO3400A, Coert-Vonk:MOSFET N-CH 30V 5.7A AO3400A SOT23-3L, symbol Coert-Vonk:MOSFET N-CH 30V 5.7A AO3400A SOT23-3L
- added R1, R12, R17, R18, R19, R21: 10k, Coert-Vonk:RES 10kΩ ±1 18W Yageo 0805, symbol Coert-Vonk:RES 10kΩ ±1% 1/8W Yageo 0805
- added R11, R13, R14, R15, R20, R3: 100Ω, Coert-Vonk:RES 100Ω ±1 18W Yageo 0805, symbol Coert-Vonk:RES 100Ω ±1% 1/8W Yageo 0805
Connections:
- net 12V: now also C6.1, HDR1.1, HDR2.1, HDR3.1, HDR4.1, HDR5.1, HDR6.1
- net 5V: now also C1.1
- net ATO_VALVE: now also R11.1
- net GND: now also C1.2, C6.2, D3.A, D4.A, D5.A, D6.A, D7.A, D9.A, Q1.2 (S), Q2.2 (S), Q3.2 (S), Q4.2 (S), Q5.2 (S), Q8.2 (S), R1.1, R12.1, R17.1, R18.1, R19.1, R21.1
- net PUMP_MAIN: now also R3.1
- net PUMP_NUT_A: now also R15.1
- net PUMP_NUT_B: now also R20.1
- net PUMP_PH_DN: now also R14.1
- net PUMP_PH_UP: now also R13.1
- new net: Q4.1 (G), R15.2, R19.2
- new net: Q1.1 (G), R1.2, R3.2
- new net: D9.C, HDR1.2, Q1.3 (D)
- new net: D3.C, HDR2.2, Q8.3 (D)
- new net: D6.C, HDR5.2, Q4.3 (D)
- new net: Q3.1 (G), R14.2, R18.2
- new net: Q2.1 (G), R13.2, R17.2
- new net: D5.C, HDR4.2, Q3.3 (D)
- new net: Q8.1 (G), R11.2, R12.2
- new net: D7.C, HDR6.2, Q5.3 (D)
- new net: Q5.1 (G), R20.2, R21.2
- new net: D4.C, HDR3.2, Q2.3 (D)
- no-connect marks 9 -> 8
Other:
- note removed: "STATUS LED"
- moved on the sheet: C4, D1, F1, J1, R4, R5, U1

Commit message: update w design and schematic
Parts:
- removed C2, C3: 100nF, Capacitor_SMD:C_0805_2012Metric, symbol Device:C
- removed J11: Float_Low, Connector_JST:JST_XH_B2B-XH-A_1x02_P2.50mm_Vertical, symbol Connector:Conn_01x02_Pin
- removed J12: BME280, Connector_JST:JST_PH_B4B-PH-K_1x04_P2.00mm_Vertical, symbol Connector:Conn_01x04_Pin
- removed J14: Float_High, Connector_JST:JST_XH_B2B-XH-A_1x02_P2.50mm_Vertical, symbol Connector:Conn_01x02_Pin
- removed J3: BH1750, Connector_JST:JST_PH_B4B-PH-K_1x04_P2.00mm_Vertical, symbol Connector:Conn_01x04_Pin
- removed J4: 1-Wire, Connector_JST:JST_PH_B3B-PH-K_1x03_P2.00mm_Vertical, symbol Connector:Conn_01x03_Pin
- removed J6: OLED, Connector_JST:JST_PH_B4B-PH-K_1x04_P2.00mm_Vertical, symbol Connector:Conn_01x04_Pin
- removed J7: HC-SR04, Connector_JST:JST_XH_B4B-XH-A_1x04_P2.50mm_Vertical, symbol Connector:Conn_01x04_Pin
- removed R2: 4.7k, Resistor_SMD:R_0805_2012Metric, symbol Device:R
- removed R6: 1k, Resistor_SMD:R_0805_2012Metric, symbol Device:R
- removed R7: 2.2k, Resistor_SMD:R_0805_2012Metric, symbol Device:R
- removed R8, R9: 10k, Resistor_SMD:R_0805_2012Metric, symbol Device:R
- added C10, C25, C27, C33: 10μF, Coert-Vonk:CAP X7R 10μF ±10 16V 0805, symbol Coert-Vonk:CAP X7R 10μF ±10% 16V 0805
- added C15, C19, C23, C26, C28, C29, C31, C34, C35, C36: 100nF, Coert-Vonk:CAP X7R 100nF ±10 25V 0805, symbol Coert-Vonk:CAP X7R 100nF ±10% 25V 0805
- added C20, C24, C30, C32: 10nF, Coert-Vonk:CAP X7R 10nF ±10% 50V 0805, symbol Coert-Vonk:CAP X7R 10nF ±10% 50V 0805
- added EZO1: EC, symbol Coert-Vonk:EVAL EZO pH
- added EZO2: DO, symbol Coert-Vonk:EVAL EZO pH
- added FB1, FB2, FB3, FB4: 330Ω at 100MHz, Coert-Vonk:FERRITE BEAD 330Ω 0805, symbol Coert-Vonk:FERRITE BEAD 330Ω 0805
- added HDR10, HDR9: Phoenix Hdr, Coert-Vonk:TERM BLOCK HDR 2POS RA 3.81mm 1803277, symbol Coert-Vonk:TERM BLOCK HDR 2POS RA 3.81mm
- added HDR7: Phoenix 45°, Coert-Vonk:TERM BLOCK HDR 1WIRE 3POS RA 3.81mm 1803280, symbol Coert-Vonk:TERM BLOCK HDR 3POS 1WIRE RA 3.81mm
- added HDR8: Phoenix 45°, Coert-Vonk:TERM BLOCK HDR 1WIRE 3POS RA 3.81mm 1803280, symbol Coert-Vonk:TERM BLOCK HDR 4POS RA 3.81mm
- added J2, J5: JST-PA, Coert-Vonk:CONN MALE 4POS RA 2mm I2C JST S04B-PASK-2, symbol Coert-Vonk:CONN I2C MALE 4POS RA 2mm JST S04B-PASK-2
- added J3, J6: BNC, Coert-Vonk:CONN BNC JACK RA 50Ω, symbol Coert-Vonk:CONN BNC JACK RA 50Ω 5227161-6
- added R10, R22: 16k9, Coert-Vonk:RES 16.9kΩ ±1 18W 0805, symbol Coert-Vonk:RES 16.9kΩ ±1% 1/8W 0805
- added R16, R29: 10k, Coert-Vonk:RES 10kΩ 0805, symbol Coert-Vonk:RES 10kΩ ±1% 1/8W 0805
- added R2, R31: 10k, Coert-Vonk:RES 10kΩ ±1 18W Yageo 0805, symbol Coert-Vonk:RES 10kΩ ±1% 1/8W Yageo 0805
- added R30: 4k7, Coert-Vonk:RES 4.7kΩ ±1 18W Yageo 0805, symbol Coert-Vonk:RES 4.7kΩ ±1% 1/8W Yageo 0805
- added U4, U5: ADM3260, Coert-Vonk:IC ISOLTR 2.5KV 2CH I2C 20SSOP ADM3260, symbol Coert-Vonk:IC ISOLTR 2.5KV 2CH I2C 20SSOP ADM3260
- HDR1: value PUMP_MAIN -> Phoenix 3.81mm
- HDR2: value ATO_VALVE -> Phoenix 3.81mm
- HDR3: value PUMP_PH_UP -> Phoenix 3.81mm
- HDR4: value PUMP_PH_DN -> Phoenix 3.81mm
- HDR5: value PUMP_NUT_A -> Phoenix 3.81mm
- HDR6: value PUMP_NUT_B -> Phoenix 3.81mm
- J15: value PH -> BNC
Connections:
- net 3V3: now also C23.2, C24.2, C25.2, C26.2, C31.2, C32.2, C33.2, C34.2, HDR7.1 (3V3), HDR8.1, J2.2 (+3V3), J5.2 (+3V3), R2.2, R30.2, R31.2, U4.4 (VDD_{P}), U4.9 (V_{IN}), U5.4 (VDD_{P}), U5.9 (V_{IN})
- net EZO_PDIS: now also U4.8 (PDIS), U5.8 (PDIS)
- net FLOAT_LOW: now also C35.2, HDR9.1, R2.1
- net GND: now also TP4.1, C23.1, C24.1, C25.1, C26.1, C31.1, C32.1, C33.1, C34.1, C35.1, C36.1, HDR10.2, HDR7.3 (GND), HDR8.4, HDR9.2, J2.1 (GND), J5.1 (GND), U4.1 (GND_{P}), U4.10 (GND_{P}), U4.5 (GND_{P}), U4.7 (GND_{P}), U5.1 (GND_{P}), U5.10 (GND_{P}), U5.5 (GND_{P}), U5.7 (GND_{P})
- net I2C_SCL: now also J2.4 (I2C_SCL), J5.4 (I2C_SCL), U4.2 (SCL_{2}), U5.2 (SCL_{2})
- net I2C_SDA: now also J2.3 (I2C_SDA), J5.3 (I2C_SDA), U4.3 (SDA_{2}), U5.3 (SDA_{2})
- net ONE_WIRE: now also HDR7.2 (DQ), R30.1
- net US_ECHO: now also HDR8.3
- net US_TRIG: now also HDR8.2
- net FLOAT_HIGH renamed ~{FLOAT_HIGH}
- net ~{FLOAT_HIGH}: now also C36.2, HDR10.1, R31.1
- new net: C15.2, C20.2, EZO1.6 (VCC), FB1.1, R10.2, U4.17 (VDD_{ISO})
- new net: C10.2, C19.2, FB1.2, U4.12 (V_{ISO})
- new net: C10.1, C15.1, C19.1, C20.1, FB2.2, R16.1, U4.11 (GND_{ISO}), U4.14 (GND_{ISO}), U4.16 (GND_{ISO}), U4.20 (GND_{ISO})
- new net: R10.1, R16.2, U4.13 (VSEL)
- new net: EZO1.3 (RX/SDA), U4.18 (SDA_{1})
- new net: EZO1.2 (TX/SCL), U4.19 (SCL_{1})
- new net: C27.1, C28.1, C29.1, C30.1, FB4.2, R29.1, U5.11 (GND_{ISO}), U5.14 (GND_{ISO}), U5.16 (GND_{ISO}), U5.20 (GND_{ISO})
- new net: R22.1, R29.2, U5.13 (VSEL)
- new net: C27.2, C29.2, FB3.2, U5.12 (V_{ISO})
- new net: EZO2.1 (GND), FB4.1
- new net: EZO2.2 (TX/SCL), U5.19 (SCL_{1})
- new net: EZO2.3 (RX/SDA), U5.18 (SDA_{1})
- new net: EZO2.4 (PGND), J6.G (GND)
- new net: EZO2.5 (PRB), J6.S
- new net: C28.2, C30.2, EZO2.6 (VCC), FB3.1, R22.2, U5.17 (VDD_{ISO})
- new net: EZO1.1 (GND), FB2.1
- new net: EZO1.4 (PGND), J3.G (GND)
- new net: EZO1.5 (PRB), J3.S
Other:
- note added: "ANGGREK 2V025-08 12VDC"
- note added: "ATO Valve"
- note added: "AUBIG DC40-1250"
- note added: "Adafruit RCWL-1601 Ultrasonic Sensor"
- note added: "Atlas Scientific Conductivity Probe K 1.0"
- note added: "Atlas Scientific Lab Grade Dissolved Oxygen Probe"
- note added: "Atlas Scientific Lab Grade pH Probe"
- note added: "Bosh BME280"
- note added: "Dissolved Oxygen Sensor (optional)"
- note added: "Electro Conductiviy Sensor"
- note added: "Flowline LH25-1101 Float Switch"
- note added: "I2C SENSORS"
- note added: "Kamoer NKP-DC-B08"
- note added: "Light Sensor (optional)"
- note added: "Main Pump"
- note added: "Nutrition-A Pump"
- note added: "Nutrition-B Pump"
- note added: "Ph Sensor"
- note added: "Ph-Dn Pump"
- note added: "Ph-Up Pump (optional)"
- note added: "Rohm BH1750"
- note added: "Sparkfun 11050 DS18B20"
- note added: "TEMPERATURE AND WATER SENSORS"
- note added: "Temp Sensor (optional)"
- note added: "Temp/Pres/Hum Sensor (optional)"
- note added: "Water Height"
- note removed: "1-WIRE / ULTRASONIC / FLOAT SWITCHES"
- note removed: "1-Wire (DS18B20)"
- note removed: "ANALOG→I2C"
- note removed: "I2C BUS"
- note removed: "ISOLATOR"
- note removed: "PH SENSOR"
- note removed: "Ultrasonic (HC-SR04)"
- moved on the sheet: C1, C11, C12, C13, C14, C16, C17, C18, C21, C22, C4, C5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

Commit message: update
Parts:
- removed HDR1, HDR2, HDR3, HDR4, HDR5, HDR6: Phoenix 3.81mm, Coert-Vonk:TERM BLOCK HDR 2POS RA 3.81mm 1803277, symbol Coert-Vonk:TERM BLOCK HDR 2POS RA 3.81mm
- removed HDR10, HDR9: Phoenix Hdr, Coert-Vonk:TERM BLOCK HDR 2POS RA 3.81mm 1803277, symbol Coert-Vonk:TERM BLOCK HDR 2POS RA 3.81mm
- removed HDR7: Phoenix 45°, Coert-Vonk:TERM BLOCK HDR 1WIRE 3POS RA 3.81mm 1803280, symbol Coert-Vonk:TERM BLOCK HDR 3POS 1WIRE RA 3.81mm
- removed HDR8: Phoenix 45°, Coert-Vonk:TERM BLOCK HDR 1WIRE 3POS RA 3.81mm 1803280, symbol Coert-Vonk:TERM BLOCK HDR 4POS RA 3.81mm
- added HDR1, HDR3, HDR7: COMBICON-MC, Coert-Vonk:TERM BLOCK HDR 1WIRE 3POS RA 3.81mm 1803280, symbol Coert-Vonk:TERM BLK HDR 4POS 3.81mm
- added J4: MKDS, Coert-Vonk:TERM BLK 3POS SCREW 3.5mm, symbol Coert-Vonk:TERM BLK SCREW 3POS 3.5mm
- added J7: MKDS, Coert-Vonk:TERM BLK 4POS SCREW 3.5mm, symbol Coert-Vonk:TERM BLK SCREW 4POS 3.5mm
- added J8, J9: MKDS, Coert-Vonk:TERM BLK 2POS SCREW 3.5mm, symbol Coert-Vonk:TERM BLK SCREW 2POS 3.5mm
- TP1: value +3V3 -> 12V
- TP2: value +5V -> 5V
- TP3: value +12V -> 3V3
- TP6: value SCL -> SCK
- TP7: value 1-Wire -> 1WIRE
Connections:
- net 12V: now also TP1.1, HDR1.1, HDR1.3, HDR3.1, HDR3.3, HDR7.1, HDR7.3
- net 3V3: now also TP3.1, J4.1 (Pin_1), J7.1 (Pin_1)
- net 5V: now also TP2.1
- net FLOAT_LOW: now also J8.1 (Pin_1)
- net GND: now also J4.3 (Pin_3), J7.4 (Pin_4), J8.2 (Pin_2), J9.2 (Pin_2)
- net I2C_SCL: now also TP6.1
- net I2C_SDA: now also TP5.1
- net ONE_WIRE: now also TP7.1, J4.2 (Pin_2)
- net US_ECHO: now also J7.3 (Pin_3)
- net US_TRIG: now also J7.2 (Pin_2)
- net ~{FLOAT_HIGH}: now also J9.1 (Pin_1)
- net at D9.C, Q1.3 (D): now also HDR1.2
- net at D3.C, Q8.3 (D): now also HDR1.4
- net at D6.C, Q4.3 (D): now also HDR3.2
- net at D5.C, Q3.3 (D): now also HDR7.2
- net at D7.C, Q5.3 (D): now also HDR3.4
- net at D4.C, Q2.3 (D): now also HDR7.4
Other:
- note added: "(2x) Kamoer NKP-DC-B08"
- note added: "ANGGREK 2V025-08"
- note added: "SoC"
- note removed: "ANGGREK 2V025-08 12VDC"
- note removed: "ESP32-C6-DevKitC"
- note removed: "Kamoer NKP-DC-B08"
- note removed: "Nutrition-B Pump"
- moved on the sheet: C35, C36, D3, D4, D5, D6, D7, D9, PCB1A, Q1, Q2, Q3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

Commit message: fix ERC errs
Parts:
- removed C11: 22μF, Coert-Vonk:CAP CER 22μF 10V 0805, symbol Coert-Vonk:CAP CER 22μF 10V 0805
- removed C27: 10μF, Coert-Vonk:CAP X7R 10μF ±10 16V 0805, symbol Coert-Vonk:CAP X7R 10μF ±10% 16V 0805
- removed C28, C29, C34: 100nF, Coert-Vonk:CAP X7R 100nF ±10 25V 0805, symbol Coert-Vonk:CAP X7R 100nF ±10% 25V 0805
- removed C30, C32: 10nF, Coert-Vonk:CAP X7R 10nF ±10% 50V 0805, symbol Coert-Vonk:CAP X7R 10nF ±10% 50V 0805
- removed C4: 10μF, Coert-Vonk:CAP CER 10µF 25V 0805, symbol Coert-Vonk:CAP CER 10µF 25V 0805
- removed C5, C8: 100nF, Coert-Vonk:CAP CER 100nF 25V 0805, symbol Coert-Vonk:CAP CER 100nF 25V 0805
- removed C7: 33nF, Coert-Vonk:CAP CER 33nF 25V 0805, symbol Coert-Vonk:CAP CER 33nF 25V 0805
- removed C9: 47μF, Coert-Vonk:CAP CER 47μF 10V 0805, symbol Coert-Vonk:CAP CER 47μF 10V 0805
- removed EZO: PH, symbol Coert-Vonk:EVAL EZO pH
- removed EZO1: EC, symbol Coert-Vonk:EVAL EZO pH
- removed EZO2: DO, symbol Coert-Vonk:EVAL EZO pH
- removed FB3, FB4: 330Ω at 100MHz, Coert-Vonk:FERRITE BEAD 330Ω 0805, symbol Coert-Vonk:FERRITE BEAD 330Ω 0805
- removed J1: JACK_5MM, Coert-Vonk:CONN JACK 2X5.5mm PJ-063AH, symbol Coert-Vonk:CONN JACK 2X5.5mm PJ-063AH
- removed J2, J5: JST-PA, Coert-Vonk:CONN MALE 4POS RA 2mm I2C JST S04B-PASK-2, symbol Coert-Vonk:CONN I2C MALE 4POS RA 2mm JST S04B-PASK-2
- removed R10, R22, R27: 16k9, Coert-Vonk:RES 16.9kΩ ±1 18W 0805, symbol Coert-Vonk:RES 16.9kΩ ±1% 1/8W 0805
- removed R16, R24, R28, R29, R4: 10k, Coert-Vonk:RES 10kΩ 0805, symbol Coert-Vonk:RES 10kΩ ±1% 1/8W 0805
- removed R23: 52k3, Coert-Vonk:RES 52.3kΩ 0805, symbol Coert-Vonk:RES 52.3kΩ ±1% 1/8W 0805
- removed R5: 100k, Coert-Vonk:RES 100kΩ 0805, symbol Coert-Vonk:RES 100kΩ ±1% 1/8W 0805
- removed U1: SI2301, Coert-Vonk:MOSFET P-CH 20V 3.1A SI2301CDS SOT23-3, symbol Coert-Vonk:MOSFET P-CH 20V 3.1A SI2301CDS SOT23-3
- removed U5: ADM3260, Coert-Vonk:IC ISOLTR 2.5KV 2CH I2C 20SSOP ADM3260, symbol Coert-Vonk:IC ISOLTR 2.5KV 2CH I2C 20SSOP ADM3260
- added C2: 47μF, Coert-Vonk:CAP X5R 47μF ±10 10V 1206, symbol Coert-Vonk:CAP X5R 47μF ±10% 10V 1206
- added C3, C5: 100nF, Coert-Vonk:CAP X7R 100nF ±10 25V 0805, symbol Coert-Vonk:CAP X7R 100nF ±10% 25V 0805
- added C4: 10μF, Coert-Vonk:CAP X7R 10μF ±10 16V 0805, symbol Coert-Vonk:CAP X7R 10μF ±10% 16V 0805
- added C7: 33nF, Coert-Vonk:CAP X7R 33nF ±10 25V 0805, symbol Coert-Vonk:CAP X7R 33nF ±10% 25V 0805
- added C8: 22μF, Coert-Vonk:CAP X7R 22μF ±10 10V 1206, symbol Coert-Vonk:CAP X7R 22μF ±10% 10V 1206
- added J1: Barrel Rcpt, Coert-Vonk:CONN JACK 2X5.5mm PJ-063AH, symbol Coert-Vonk:CONN JACK RCPT 2X5.5mm PJ-063AH
- added J2, J5: JST_PH, Coert-Vonk:HEADER MALE 4POS 2mm JST-PA, symbol Coert-Vonk:HEADER MALE 4POS 2mm JST-PH
- added MEZZ1: RTD, Coert-Vonk:MEZZ EZO RTD, symbol Coert-Vonk:MEZZ_EZO_RTD
- added MEZZ2: EC, Coert-Vonk:MEZZ EZO EC, symbol Coert-Vonk:MEZZ EZO EC
- added MEZZ3: pH, Coert-Vonk:MEZZ EZO pH, symbol Coert-Vonk:MEZZ EZO pH
- added R10, R7: 16k9, Coert-Vonk:RES 16.9kΩ ±1 18W 0805, symbol Coert-Vonk:RES 16.9kΩ ±1% 1/8W Yageo 0805
- added R16, R4, R6, R9: 10k, Coert-Vonk:RES 10kΩ ±1 18W Yageo 0805, symbol Coert-Vonk:RES 10kΩ ±1% 1/8W Yageo 0805
- added R5: 100k, Coert-Vonk:RES 100kΩ 0805, symbol Coert-Vonk:RES 100kΩ ±1% 1/8W Yageo 0805
- added R8: 52k3, Coert-Vonk:RES 52.3kΩ 0805, symbol Coert-Vonk:RES 52.3kΩ ±1% 1/8W Yageo 0805
- added U1: SI2301, Coert-Vonk:MOSFET P-CH 20V 3.1A SI2301CDS SOT23-3, symbol Coert-Vonk:MOSFET P-CH 20V 3.1A SI2301 SOT23-3
- R25, R26: footprint Coert-Vonk:RES 4.7kΩ 0805 -> Coert-Vonk:RES 4.7kΩ ±1 18W Yageo 0805; symbol Coert-Vonk:RES 4.7kΩ ±5% 1/4W 0805 -> Coert-Vonk:RES 4.7kΩ ±1% 1/8W Yageo 0805; DKPN 738-RMCA0805JT4K70-HPCT-ND -> 311-4.70KCRCT-ND
Connections:
- net 12V: now also C4.2, C5.2, U1.3 (D)
- net 3V3: now also C8.2, J2.2 (3V3), J5.2 (3V3), MEZZ1.6 (VCC)
- net 5V: now also C2.2, R8.2
- net GND: now also C2.1, C4.1, C5.1, C7.1, C8.1, J1.2, J1.S (SHIELD), J1.S2 (SHIELD__1), J2.1 (GND), J5.1 (GND), MEZZ1.1 (GND), R5.1, R9.1
- net I2C_SCL: now also J2.4 (I2C_SCL), J5.4 (I2C_SCL), MEZZ1.2 (TX/SCL)
- net I2C_SDA: now also J2.3 (I2C_SDA), J5.3 (I2C_SDA), MEZZ1.3 (RX/SDA)
- net at C15.2, C20.2, FB1.1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: now also MEZZ2.6 (VCC), R10.2
- net at L1.1, U2.5 (SW): now also C3.2
- net at U3.13 (VSEL): now also R6.1, R7.1
- net at C16.2, C18.2, FB8.1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: now also MEZZ3.6 (VCC), R7.2
- net at C10.1, C15.1, C19.1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: now also R16.2
- net at U4.13 (VSEL): now also R10.1, R16.1
- net at U4.18 (SDA_{1}): now also MEZZ2.3 (RX/SDA)
- net at U4.19 (SCL_{1}): now also MEZZ2.2 (TX/SCL)
- net at C13.1, C14.1, C16.1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: now also R6.2
- net at U2.8 (FB): now also R8.1, R9.2
- net at F1.1: now also J1.1
- net at FB7.1: now also MEZZ3.1 (GND)
- net at U3.19 (SCL_{1}): now also MEZZ3.2 (TX/SCL)
- net at U3.18 (SDA_{1}): now also MEZZ3.3 (RX/SDA)
- net at J15.G (GND): now also MEZZ3.4 (PGND)
- net at J15.S: now also MEZZ3.5 (PRB)
- net at J6.G (GND): now also MEZZ1.4 (PGND)
- net at J6.S: now also MEZZ1.5 (PRB)
- net at FB2.1: now also MEZZ2.1 (GND)
- net at J3.G (GND): now also MEZZ2.4 (PGND)
- net at J3.S: now also MEZZ2.5 (PRB)
- net at D1.1 (C), F1.2: now also R4.2, U1.2 (S)
- net at U2.6 (BST): now also C3.1
- net at U2.7 (SS): now also C7.2
- new net: R4.1, R5.2, U1.1 (G)
- no-connect marks 8 -> 14
Other:
- note added: "Environmental Sensor (optional)"
- note added: "Temperature Sensor (optional)"
- note removed: "Dissolved Oxygen Sensor (optional)"
- note removed: "Temp/Pres/Hum Sensor (optional)"
- moved on the sheet: C31, C33
