File: hardware/OPNhydro_r1/OPNhydro_r1.kicad_sch (KiCad schematic)
At the start: 101 parts, among them J1 Barrel Rcpt, J15 BNC, J2 JST_PH, J3 BNC, J4 MKDS, J5 JST_PH, J6 BNC, J7 MKDS, J8 MKDS, J9 MKDS, Q1 2N7002K, Q2 AO3400A, Q3 AO3400A, Q4 AO3400A, Q5 AO3400A, Q8 AO3400A, U1 SI2301, U2 TPS62933, U3 ADM3260, U4 ADM3260

Commit message: ùpdate
Parts:
- removed C1: 1000μF, Coert-Vonk:CAP ALUM POLY 1000μF ±20 6.3V, symbol Coert-Vonk:CAP ALUM POLY 1000μF ±20% 6.3V
- removed D7, D9: SS34, Coert-Vonk:DIODE SCHOTTKY 40V 3A DIOM7959X265N DO214AB, symbol Coert-Vonk:DIODE SCHOTTKY 40V 3A DIOM7959X265N DO214AB
- removed HDR1, HDR3, HDR7: COMBICON-MC, Coert-Vonk:TERM BLOCK HDR 1WIRE 3POS RA 3.81mm 1803280, symbol Coert-Vonk:TERM BLK HDR 4POS 3.81mm
- removed J2, J5: JST_PH, Coert-Vonk:HEADER MALE 4POS 2mm JST-PA, symbol Coert-Vonk:HEADER MALE 4POS 2mm JST-PH
- removed J4: MKDS, Coert-Vonk:TERM BLK 3POS SCREW 3.5mm, symbol Coert-Vonk:TERM BLK SCREW 3POS 3.5mm
- removed L1: 7.8µH, Coert-Vonk:IND 7.8µH 10A 20.5mΩ, symbol Coert-Vonk:IND 7.8µH 10A 20.5mΩ
- removed Q1: 2N7002K, Coert-Vonk:MOSFET N-CH 55V 42A IRLR2905TRPBF DPAK, symbol Coert-Vonk:MOSFET N-CH 55V 42A IRLR2905TRPBF DPAK
- removed Q2, Q3, Q4: AO3400A, Coert-Vonk:MOSFET N-CH 30V 5.7A AO3400A SOT23-3L, symbol Coert-Vonk:MOSFET N-CH 30V 5.7A AO3400A SOT23-3L
- removed R13, R14: 100Ω, Coert-Vonk:RES 100Ω ±1 18W Yageo 0805, symbol Coert-Vonk:RES 100Ω ±1% 1/8W Yageo 0805
- removed R17, R18: 10k, Coert-Vonk:RES 10kΩ ±1 18W Yageo 0805, symbol Coert-Vonk:RES 10kΩ ±1% 1/8W Yageo 0805
- removed R30: 4k7, Coert-Vonk:RES 4.7kΩ ±1 18W Yageo 0805, symbol Coert-Vonk:RES 4.7kΩ ±1% 1/8W Yageo 0805
- added C9: 1000μF, Coert-Vonk:CAP ALUM 1000μF ±20 10V, symbol Coert-Vonk:CAP ALUM 1000μF ±20% 10V
- added D2: SS34, Coert-Vonk:DIODE SCHOTTKY 40V 3A DIOM7959X265N DO214AB, symbol Coert-Vonk:DIODE SCHOTTKY 40V 3A DIOM7959X265N DO214AB
- added HDR4, HDR5: JST_PH, Coert-Vonk:HEADER MALE 4POS 2mm JST-PA, symbol Coert-Vonk:TERM BLK HDR 4POS JST-PH 2mm
- added HDR6: MC_0.2", Coert-Vonk:TERM BLK HDR 2POS 5.08mm, symbol Coert-Vonk:TERM BLK HDR 2POS 5.08mm
- added HDR7: MC_0.15", Coert-Vonk:TERM BLK HDR 6POS 3.81mm, symbol Coert-Vonk:TERM BLK HDR 6POS 3.81mm
- added HDR8: MC_0.15", Coert-Vonk:TERM BLK HDR 2POS 3.81mm, symbol Coert-Vonk:TERM BLK HDR 2POS 3.81mm
- added L1: 5.6µH, Coert-Vonk:IND 5.6µH 3.5A 40mΩ, symbol Coert-Vonk:IND 5.6µH 3.5A 40mΩ
- added P1: MAIN, symbol Coert-Vonk:PUMP AUBIG DC40-1250
- added P2: PH↓, symbol Coert-Vonk:PUMP KAMOER NKP-DC-B08
- added P3: NUT_A, symbol Coert-Vonk:PUMP KAMOER NKP-DC-B08
- added P4: NUT_B, symbol Coert-Vonk:PUMP KAMOER NKP-DC-B08
- added PB1: USS, symbol Coert-Vonk:PROBE ULTRASONIC SENSOR
- added PB2: pH, symbol Coert-Vonk:PROBE ATLAS ENV-40-PH
- added PB3: EC_K1.0, symbol Coert-Vonk:PROBE ATLAS ENV-40-EC-K1.0
- added PB4: RTD, symbol Coert-Vonk:PROBE ATLAS PT-1000
- added PB5, PB6: BME280, symbol Coert-Vonk:PROBE BOSCH BME280
- added PLG1, PLG2: PHR-4, symbol Coert-Vonk:TERM BLK PLG 4POS JST-PH 2mm
- added PLG3: MC_0.2", Coert-Vonk:TERM BLK PLUG 2POS 5.08mm, symbol Coert-Vonk:TERM BLK PLUG 2POS 5.08mm
- added PLG4: MC_0.15", Coert-Vonk:TERM BLK PLUG 6POS 3.81mm, symbol Coert-Vonk:TERM BLK PLG 6POS 3.81mm
- added PLG5: MC_0.15", Coert-Vonk:TERM BLOCK PLUG 2POS 3.81mm 1803578, symbol Coert-Vonk:TERM BLK PLG 2POS 3.81mm
- added R14, R21: 4k7, Coert-Vonk:RES 4.7kΩ ±1 18W Yageo 0805, symbol Coert-Vonk:RES 4.7kΩ ±1% 1/8W Yageo 0805
- added R16: 10k, Coert-Vonk:RES 10kΩ ±1 18W Yageo 0805, symbol Coert-Vonk:RES 10kΩ ±1% 1/8W Yageo 0805
- added R18: 100Ω, Coert-Vonk:RES 100Ω ±1 18W Yageo 0805, symbol Coert-Vonk:RES 100Ω ±1% 1/8W Yageo 0805
- added SW1, SW2: FLOAT, symbol Coert-Vonk:SWITCH FLOAT
- added T2, T6: BT3904, Coert-Vonk:TRANS NPN 40V 0.2A SOT23-3, symbol Coert-Vonk:TRANS NPN 40V 0.2A SOT23-3
- added T3, T5: AO3400A, Coert-Vonk:MOSFET N-CH 30V 5.7A AO3400A SOT23-3L, symbol Coert-Vonk:MOSFET N-CH 30V 5.7A AO3400A SOT23-3L
- added T4: IRLR2905, Coert-Vonk:MOSFET N-CH 55V 42A IRLR2905TRPBF DPAK, symbol Coert-Vonk:MOSFET N-CH 55V 42A IRLR2905 DPAK
- added V1: ATO, symbol Coert-Vonk:VALVE ANGGREK 2V025-08
- TP1: value 12V -> TestPoint
- TP2: value 5V -> TestPoint
- TP3: value 3V3 -> TestPoint
- TP4: value GND -> TestPoint
- TP5: value SDA -> TestPoint
- TP6: value SCK -> TestPoint
- TP7: value 1WIRE -> TestPoint
- renumbered C35 to C1, C31 to C10, C14 to C11, C16 to C12, C10 to C13, C15 to C14, C33 to C15, C13 to C16, C18 to C17, C19 to C18, C20 to C19, C6 to C2, C8 to C20, C12 to C21, C17 to C25, C21 to C26, C25 to C27, C26 to C28, C36 to C3, C7 to C6, C3 to C7, C2 to C8, FB8 to FB1, FB7 to FB2, FB1 to FB3, FB2 to FB4, J7 to HDR1, J8 to HDR2, J9 to HDR3, J15 to J2, J6 to J4, MEZZ3 to MEZZ1, MEZZ1 to MEZZ3, R26 to R1, R6 to R11, R16 to R12, R3 to R13, R1 to R17, R25 to R2, R11 to R20, R20 to R22, R21 to R23, R12 to R24, R2 to R3, R31 to R6, R8 to R7, R9 to R8, R7 to R9, U1 to T1, Q5 to T7, Q8 to T8, U2 to U1, U3 to U2, U4 to U3
Connections:
- net 12V: now also D3.C, D4.C, D5.C, D6.C, D2.C, HDR6.1, HDR7.1, HDR7.3, HDR7.5, HDR8.1
- net 3V3: now also C3.2, HDR3.1 (Pin_1), HDR4.2 (3V3), HDR5.2 (3V3); no longer R6.2
- net 5V: now also C9.1, L1.2
- net FLOAT_LOW: now also R21.1
- net GND: now also R6.1, C9.2, HDR4.1 (GND), HDR5.1 (GND), R16.1, T2.2 (E), T3.2 (S), T4.2 (S), T5.2 (S), T6.2 (E); no longer C3.1, D3.A, D4.A, D5.A, D6.A, HDR3.2 (Pin_2)
- net I2C_SCL: now also HDR4.4 (I2C_SCL), HDR5.4 (I2C_SCL)
- net I2C_SDA: now also HDR4.3 (I2C_SDA), HDR5.3 (I2C_SDA)
- net PUMP_NUT_A: now also R18.2; no longer R15.1
- net PUMP_NUT_B: now also R22.2; no longer R22.1
- net PUMP_PH_DN: now also R15.2
- net at R19.2: now also R18.1, T5.1 (G); no longer R15.2
- net at C7.2, U1.5 (SW): now also L1.1
- net at R13.2, R17.2: now also T2.3 (C), T4.1 (G)
- net at T8.3 (D): now also D6.A, HDR8.2; no longer D3.C
- net 0V8: now reaches R7.1, R8.2, U1.8 (FB)
- net at R20.2, R24.2, T8.1 (G): now also T6.3 (C)
- net at T7.3 (D): now also D5.A, HDR7.6
- net at R23.2, T7.1 (G): now also R22.1; no longer R22.2
- removed net ~{FLOAT_HIGH}: C3.2, HDR3.1 (Pin_1), PCB1.J1_8 (IO1/ADC1), R6.1
- new net: R15.1, R16.2, T3.1 (G)
- new net: D2.A, HDR7.2, T3.3 (D)
- new net: R14.2, T2.1 (B)
- new net: D3.A, HDR6.2, T4.3 (D)
- new net: R21.2, T6.1 (B)
- new net: P1.12V, PLG3.1
- new net: P1.GND, PLG3.2
- new net: PB6.1, PLG2.1
- new net: PB6.2, PLG2.2
- new net: PB6.3, PLG2.3
- new net: PB6.4, PLG2.4
- new net: PLG5.1, V1.12V
- new net: PLG5.2, V1.GND
- new net: P4.12V, PLG4.5
- new net: P4.GND, PLG4.6
- new net: PB5.1, PLG1.1
- new net: PB5.2, PLG1.2
- new net: PB5.3, PLG1.3
- new net: PB5.4, PLG1.4
- new net: D4.A, HDR7.4, T5.3 (D)
- new net: P2.12V, PLG4.1
- new net: P2.GND, PLG4.2
- new net: P3.12V, PLG4.3
- new net: P3.GND, PLG4.4
- new net FLOAT_HIGH: C3.1, HDR3.2 (Pin_2), PCB1.J1_8 (IO1/ADC1), R14.1, R6.2
Other:
- note added: "5ms soft-start"
- note added: "Bootstrap"
- note added: "Bulk for motor surge"
- note added: "Bulk for radio TX"
- note added: "Float High Switch"
- note added: "Float Low Switch"
- note added: "Flyback"
- note added: "Noise mitigation"
- note added: "Nutition Pumps"
- note added: "PUMP & VALVE DRIVERS"
- note added: "Ph↓ Pump"
- note added: "Prevent high-frequency oscillation"
- note added: "Stay off during SoC reset"
- note added: "WATER LEVEL SENSORS"
- note added: "Water Height Sensor"
- note added: "Water Temperature Sensor"
- note removed: "(2x) Kamoer NKP-DC-B08"
- note removed: "ANGGREK 2V025-08"
- note removed: "AUBIG DC40-1250"
- note removed: "Adafruit RCWL-1601 Ultrasonic Sensor"
- note removed: "Atlas Scientific Conductivity Probe K 1.0"
- note removed: "Atlas Scientific Lab Grade Dissolved Oxygen Probe"
- note removed: "Atlas Scientific Lab Grade pH Probe"
- note removed: "Bosh BME280"
- note removed: "Float Switches"
- note removed: "Flowline LH25-1101 Float Switch"
- note removed: "Nutrition-A Pump"
- note removed: "PUMP & VALVE DRIVERS (12V)"
- note removed: "Ph-Dn Pump"
- note removed: "Ph-Up Pump (optional)"
- note removed: "Rohm BH1750"
- note removed: "Sparkfun 11050 DS18B20"
- note removed: "TEMPERATURE AND WATER SENSORS"
- note removed: "Temp Sensor (optional)"
- note removed: "Temperature Sensor (optional)"
- note removed: "Water Height"
- company: (none) -> https://github.com/cvonk/OPNhydro
- title: (none) -> OPNhydro
- moved on the sheet: C1, C10, C15, C3, HDR1, HDR2, J2, J3, J4, MEZZ1, MEZZ2, MEZZ3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

Commit message: fix erc errs
Parts:
- removed PLG3: MC_0.2", Coert-Vonk:TERM BLK PLUG 2POS 5.08mm, symbol Coert-Vonk:TERM BLK PLUG 2POS 5.08mm
- added PLG6: MC_0.2", Coert-Vonk:TERM BLK PLUG 2POS 5.08mm, symbol Coert-Vonk:TERM BLK PLG 2POS 5.08mm
- P2: value PH↓ -> pH↓
Connections:
- net at P1.12V: now also PLG6.1
- net at P1.GND: now also PLG6.2
- net PUMP_PH_UP: no longer names the net of PCB1.J1_11 (IO11)
- new net: PB3.G, PB3.S
- no-connect marks 14 -> 15
Changed lines of the file:
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@@
 	)
 	(junction
-		(at 392.43 102.87)
-		(diameter 0)
-		(color 0 0 0 0)
-	)
-	(junction
 		(at 240.03 196.85)
 		(diameter 0)
@@
 	)
 	(junction
-		(at 392.43 100.33)
-		(diameter 0)
-		(color 0 0 0 0)
-	)
-	(junction
 		(at 209.55 38.1)
 		(diameter 0)
@@
 	)
 	(no_connect
+		(at 92.71 110.49)
+	)
+	(no_connect
 		(at 92.71 125.73)
 	)
@@
 	(wire
 		(pts
-			(xy 392.43 102.87) (xy 394.97 102.87)
-		)
-		(stroke
-			(width 0)
-			(type default)
-		)
-	)
-	(wire
-		(pts
 			(xy 254 139.7) (xy 254 149.86)
 		)
@@
 	(wire
 		(pts
-			(xy 92.71 110.49) (xy 95.25 110.49)
-		)
-		(stroke
-			(width 0)
-			(type default)
-		)
-	)
-	(wire
-		(pts
 			(xy 105.41 58.42) (xy 105.41 62.23)
 		)
@@
 	(wire
 		(pts
-			(xy 392.43 100.33) (xy 394.97 100.33)
-		)
-		(stroke
-			(width 0)
-			(type default)
-		)
-	)
-	(wire
-		(pts
 			(xy 199.39 222.25) (xy 199.39 220.98)
 		)
@@
 		)
 	)
-	(global_label "PUMP_PH_UP"
-		(shape output)
-		(at 95.25 110.49 0)
-		(fields_autoplaced yes)
-		(effects
-			(font
-				(size 1.27 1.27)
-			)
-			(justify left)
-		)
-		(property "Intersheetrefs" "${INTERSHEET_REFS}"
-			(at 108.6976 110.49 0)
-			(effects
-				(font
-					(size 1.27 1.27)
-				)
-				(justify left)
-				(hide yes)
-			)
-		)
-	)
 	(global_label "I2C_SDA"
 		(shape bidirectional)
@@
 	)
 	(symbol
-		(lib_id "Coert-Vonk:TERM BLK PLUG 2POS 5.08mm")
-		(at 326.39 97.79 0)
-		(mirror y)
-		(unit 1)
-		(exclude_from_sim no)
-		(in_bom yes)
-		(on_board no)
-		(dnp no)
-		(property "Reference" "PLG3"
-			(at 326.39 107.696 0)
-			(effects
-				(font
-					(size 1.27 1.27)
-				)
-			)
-		)
-		(property "Value" "MC_0.2\""
-			(at 326.39 110.236 0)
-			(effects
-				(font
-					(size 1.27 1.27)
-				)
-			)
-		)
-		(property "Footprint" "Coert-Vonk:TERM BLK PLUG 2POS 5.08mm"
-			(at 326.39 97.79 0)
-			(effects
-				(font
-					(size 1.27 1.27)
-					(italic yes)
-				)
-				(hide yes)
-			)
-		)
-		(property "Datasheet" "https://mm.digikey.com/Volume0/opasdata/d220001/medias/docus/540/1836079.pdf"
-			(at 326.39 97.79 0)
-			(effects
-				(font
-					(size 1.27 1.27)
-					(italic yes)
-				)
-				(hide yes)
-			)
-		)
-		(property "Description" "2 Position Terminal Block Plug, Female Sockets 0.200\" (5.08mm) 180° Free Hanging (In-Line)"
-			(at 326.39 97.79 0)
-			(effects
-				(font
-					(size 1.27 1.27)
-				)
-				(hide yes)
-			)
-		)
-		(property "DKPN" "277-6146-ND"
-			(at 326.39 97.79 0)
-			(effects
-				(font
-					(size 1.27 1.27)
-				)
-				(hide yes)
-			)
-		)
-		(pin "2"
-		)
-		(pin "1"
-		)
-		(instances
-			(project ""
-				(path "/a0000000-0000-4000-8000-000000002687"
-					(reference "PLG3")
-					(unit 1)
-				)
-			)
-		)
-	)
-	(symbol
 		(lib_id "Coert-Vonk:REG 3.3V 1A LDO AZ1117-3.3")
 		(at 193.04 35.56 0)
@@
 			)
 		)
-		(property "Description" ""
+		(property "Description" "Adafruit RCWL-1601 Ultrasonic Sensor"
 			(at 35.56 220.98 0)
 			(effects
@@
 			)
 		)
+		(pin "3"
+		)
+		(pin "4"
+		)
+		(pin "2"
+		)
+		(pin "1"
+		)
 		(instances
 			(project ""
@@
 	)
 	(symbol
+		(lib_name "PUMP KAMOER NKP-DC-B08_1")
 		(lib_id "Coert-Vonk:PUMP KAMOER NKP-DC-B08")
 		(at 394.97 143.51 0)
@@
 		(dnp no)
 		(property "Reference" "P2"
-			(at 395.478 152.908 0)
+			(at 394.97 138.43 0)
 			(effects
 				(font
@@
 			)
 		)
-		(property "Value" "PH↓"
-			(at 395.478 155.448 0)
+		(property "Value" "pH↓"
+			(at 394.97 140.97 0)
 			(effects
 				(font
@@
 		)
 		(instances
-			(project ""
+			(project "OPNhydro_r1"
 				(path "/a0000000-0000-4000-8000-000000002687"
 					(reference "V1")
@@
 			)
 		)
+		(pin "G"
+		)
+		(pin "S"
+		)
 		(instances
 			(project ""
@@
 					(unit 1)
 				)
+			)
+		)
+	)
+	(symbol
+		(lib_id "Coert-Vonk:TERM BLK PLG 2POS 5.08mm")
+		(at 326.39 97.79 0)
+		(mirror y)
+		(unit 1)
+		(exclude_from_sim no)
+		(in_bom yes)
+		(on_board no)
+		(dnp no)
+		(property "Reference" "PLG6"
+			(at 326.644 107.188 0)
+			(effects
+				(font
+					(size 1.27 1.27)
+				)
+			)
+		)
+		(property "Value" "MC_0.2\""
+			(at 326.644 109.728 0)
+			(effects
+				(font
+					(size 1.27 1.27)
+				)
+			)
+		)
+		(property "Footprint" "Coert-Vonk:TERM BLK PLUG 2POS 5.08mm"
+			(at 326.39 97.79 0)
+			(effects
+				(font
+					(size 1.27 1.27)
+					(italic yes)
+				)
+				(hide yes)
+			)
+		)
+		(property "Datasheet" "https://mm.digikey.com/Volume0/opasdata/d220001/medias/docus/540/1836079.pdf"
+			(at 326.39 97.79 0)
+			(effects
+				(font
+					(size 1.27 1.27)
+					(italic yes)
+				)
+				(hide yes)
+			)
+		)
+		(property "Description" "2 Position Terminal Block Plug, Female Sockets 0.200\" (5.08mm) 180° Free Hanging (In-Line)"
+			(at 326.39 97.79 0)
+			(effects
+				(font
+					(size 1.27 1.27)
+				)
+				(hide yes)
+			)
+		)
+		(property "DKPN" "277-6146-ND"
+			(at 326.39 97.79 0)
+			(effects
+				(font
+					(size 1.27 1.27)
+				)
+				(hide yes)
+			)
+		)
+		(pin "1"
+		)
+		(pin "2"
+		)
+		(instances
+			(project ""
+				(path "/a0000000-0000-4000-8000-000000002687"
+					(reference "PLG6")
+					(unit 1)
+				)

Commit message: update
Parts:
- removed HDR1: MKDS, Coert-Vonk:TERM BLK 4POS SCREW 3.5mm, symbol Coert-Vonk:TERM BLK SCREW 4POS 3.5mm
- removed HDR2, HDR3: MKDS, Coert-Vonk:TERM BLK 2POS SCREW 3.5mm, symbol Coert-Vonk:TERM BLK SCREW 2POS 3.5mm
- removed HDR4, HDR5: JST_PH, Coert-Vonk:HEADER MALE 4POS 2mm JST-PA, symbol Coert-Vonk:TERM BLK HDR 4POS JST-PH 2mm
- removed HDR6: MC_0.2", Coert-Vonk:TERM BLK HDR 2POS 5.08mm, symbol Coert-Vonk:TERM BLK HDR 2POS 5.08mm
- removed HDR7: MC_0.15", Coert-Vonk:TERM BLK HDR 6POS 3.81mm, symbol Coert-Vonk:TERM BLK HDR 6POS 3.81mm
- removed HDR8: MC_0.15", Coert-Vonk:TERM BLK HDR 2POS 3.81mm, symbol Coert-Vonk:TERM BLK HDR 2POS 3.81mm
- removed MEZZ3: RTD, Coert-Vonk:MEZZ EZO RTD, symbol Coert-Vonk:MEZZ_EZO_RTD
- removed PCB1: ESP32-C6-DEVKIT, Coert-Vonk:EVAL ESP32-C6-DEVKITC, symbol Coert-Vonk:EVAL ESP32-C6-DEVKITC-1-N8
- removed PLG1, PLG2: PHR-4, symbol Coert-Vonk:TERM BLK PLG 4POS JST-PH 2mm
- removed PLG4: MC_0.15", Coert-Vonk:TERM BLK PLUG 6POS 3.81mm, symbol Coert-Vonk:TERM BLK PLG 6POS 3.81mm
- removed PLG5: MC_0.15", Coert-Vonk:TERM BLOCK PLUG 2POS 3.81mm 1803578, symbol Coert-Vonk:TERM BLK PLG 2POS 3.81mm
- removed PLG6: MC_0.2", Coert-Vonk:TERM BLK PLUG 2POS 5.08mm, symbol Coert-Vonk:TERM BLK PLG 2POS 5.08mm
- removed SW1: FLOAT, symbol Coert-Vonk:SWITCH FLOAT
- removed TP7: TestPoint, TestPoint:TestPoint_Pad_1.0x1.0mm, symbol Connector:TestPoint
- added H1, H2: JST_PH, Coert-Vonk:HEADER MALE 4POS 2mm JST-PA, symbol Coert-Vonk:TERM BLK HDR 4POS JST-PH 2mm
- added H3: MC_0.2", Coert-Vonk:TERM BLK HDR 2POS 5.08mm, symbol Coert-Vonk:TERM BLK HDR 2POS MC 5.08mm
- added H4: MC_0.15", Coert-Vonk:TERM BLK HDR 6POS 3.81mm, symbol Coert-Vonk:TERM BLK HDR 6POS MC 3.81mm
- added H5: MC_0.15", Coert-Vonk:TERM BLK HDR 2POS 3.81mm, symbol Coert-Vonk:TERM BLK HDR 2POS MC 3.81mm
- added J1, J3: MKDS, Coert-Vonk:TERM BLK 4POS SCREW 3.5mm, symbol Coert-Vonk:TERM BLK SCREW 4POS MKDS 3.5mm
- added M1: ESP32-C6-DEVKIT, Coert-Vonk:EVAL ESP32-C6-DEVKITC, symbol Coert-Vonk:EVAL ESP32-C6-DEVKITC-1-N8
- added M4: RTD, Coert-Vonk:MEZZ EZO RTD, symbol Coert-Vonk:MEZZ EZO RTD
- added P1, P2: PHR-4, symbol Coert-Vonk:TERM BLK PLG 4POS JST-PH 2mm
- added P3: MC_0.2", Coert-Vonk:TERM BLK PLUG 2POS 5.08mm, symbol Coert-Vonk:TERM BLK PLG 2POS MC 5.08mm
- added P5: MC_0.15", Coert-Vonk:TERM BLK PLUG 6POS 3.81mm, symbol Coert-Vonk:TERM BLK PLG 6POS MC 3.81mm
- added P6: MC_0.15", Coert-Vonk:TERM BLOCK PLUG 2POS 3.81mm 1803578, symbol Coert-Vonk:TERM BLK PLG 2POS MC 3.81mm
- added SW2: FLOAT, symbol Coert-Vonk:SWITCH FLOAT LOW
- SW1: renamed from SW2; symbol Coert-Vonk:SWITCH FLOAT -> Coert-Vonk:SWITCH FLOAT HIGH
- renumbered C15 to C10, C9 to C15, C3 to C2, C2 to C3, C10 to C9, J1 to J2, J2 to J4, J3 to J5, J4 to J6, MEZZ1 to M2, MEZZ2 to M3, P1 to P4, P2 to P7, P3 to P8, P4 to P9, R4 to R3, R5 to R4, R3 to R5
Connections:
- net 12V: now also H3.1, H4.1, H4.3, H4.5, H5.1
- net 3V3: now also H1.2 (3V3), H2.2 (3V3), J1.1 (Pin_1), J3.1 (Pin_1), M4.6 (VCC)
- net 5V: now also M1.J1_14 (5V0)
- net ATO_VALVE: now also M1.J1_12 (IO2/SPI_MISO)
- net EZO_PDIS: now also M1.J1_5 (IO6/SPI_CLK)
- net FLOAT_HIGH: now also J3.2 (Pin_2), M1.J1_8 (IO1/ADC1)
- net FLOAT_LOW: now also J3.3 (Pin_3), M1.J1_7 (IO0/ADC0)
- net GND: now also H1.1 (GND), H2.1 (GND), J1.4 (Pin_4), J3.4 (Pin_4), M1.J1_15 (GND), M1.J3_1 (GND), M1.J3_12 (GND), M1.J3_15 (GND), M4.1 (GND)
- net I2C_SCL: now also H1.4 (I2C_SCL), H2.4 (I2C_SCL), M1.J1_4 (IO5/I2C_SCL), M4.2 (TX/SCL)
- net I2C_SDA: now also H1.3 (I2C_SDA), H2.3 (I2C_SDA), M1.J1_3 (IO4/I2C_SDA), M4.3 (RX/SDA)
- net PUMP_MAIN: now also M1.J1_10 (IO10)
- net PUMP_NUT_A: now also M1.J3_4 (IO15)
- net PUMP_NUT_B: now also M1.J3_9 (IO19)
- net PUMP_PH_DN: now also M1.J1_11 (IO11)
- net US_ECHO: now also J1.3 (Pin_3), M1.J1_13 (IO3/ADC3)
- net US_TRIG: now also J1.2 (Pin_2), M1.J1_6 (IO7/SPI_MOSI)
- net at FB4.1, M3.1 (GND): now also C14.2, C19.2, FB3.1, M3.6 (VCC), R10.2, U3.17 (VDD_{ISO})
- net at D2.A, T3.3 (D): now also H4.2
- net at D3.A, T4.3 (D): now also H3.2
- net at C12.2, C17.2, FB1.1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: now also FB2.1, M2.1 (GND)
- net at P4.12V: now also P3.1
- net at P4.GND: now also P3.2
- net at D6.A, T8.3 (D): now also H5.2
- net at PB6.1: now also P2.1
- net at PB6.2: now also P2.2
- net at PB6.3: now also P2.3
- net at PB6.4: now also P2.4
- net at V1.12V: now also P6.1
- net at V1.GND: now also P6.2
- net at P9.12V: now also P5.5
- net at P9.GND: now also P5.6
- net at PB5.1: now also P1.1
- net at PB5.2: now also P1.2
- net at PB5.3: now also P1.3
- net at PB5.4: now also P1.4
- net at D4.A, T5.3 (D): now also H4.4
- net at D5.A, T7.3 (D): now also H4.6
- net at J6.G (GND): now also M4.4 (PGND)
- net at J6.S: now also M4.5 (PRB)
- net at P7.12V: now also P5.1
- net at P7.GND: now also P5.2
- net at P8.12V: now also P5.3
- net at P8.GND: now also P5.4
Other:
- note added: "Safety Switches"
- note added: "WATER LEVEL SENSOR/SWITCHES"
- note added: "pH Sensor"
- note removed: "Dual function pin considerations: IO8 is used for RGB LED on the DevKitC => reserved. IO9 has internal ~45kΩ pullup. US_TRIG is a non-critical output, initialized after boot => OK. IO15 has a 10kΩ pulldown due to the MOSFET driver. This will disable ESP32 ROM boot messages. IO17 is driven by the CP2102N UART TX output => reserved. D+/D- are used for Serial Logging, Code Upload and JTAG debugging.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"
- note removed: "Float High Switch"
- note removed: "Float Low Switch"
- note removed: "Ph Sensor"
- note removed: "WATER LEVEL SENSORS"
- moved on the sheet: C1, C10, C11, C12, C13, C14, C16, C17, C18, C19, C2, C21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
