File: hardware/OPNhydro_r1/OPNhydro_r1.kicad_sch (KiCad schematic)
At the start: 115 parts, among them J1 MKDS, J2 Barrel Rcpt, J3 MKDS, J4 BNC, J5 BNC, J6 BNC, M1 ESP32-C6-DEVKIT, M2 pH, M3 EC, M4 RTD, P1 PHR-4, P2 PHR-4, P3 MC_0.2", P4 MAIN, P5 MC_0.15", P6 MC_0.15", P7 pH↓, P8 NUT_A, P9 NUT_B, SW1 FLOAT, SW2 FLOAT, T1 SI2301, T2 BT3904, T3 AO3400A, T4 IRLR2905, T5 AO3400A, T6 BT3904, T7 AO3400A, T8 AO3400A, U1 TPS62933, U2 ADM3260, U3 ADM3260

Commit message: moving to stepper motors. schematic not yet.  mark down already.
Parts:
- removed J2: Barrel Rcpt, Coert-Vonk:CONN JACK 2X5.5mm PJ-063AH, symbol Coert-Vonk:CONN JACK RCPT 2X5.5mm PJ-063AH
- removed PB5: BME280, symbol Coert-Vonk:PROBE BOSCH BME280
- added DC1: 12V/6A, symbol Coert-Vonk:SUPPLY DC 12V 72W
- added H7: MSTBA_0.2", Coert-Vonk:TERM BLK HDR 2POS MSTBA 5.08mm, symbol Coert-Vonk:TERM BLK HDR 2POS MSTBA 5.08mm
- added P10: MSTB_0.2", Coert-Vonk:TERM BLK PLG 2POS MSTB 5.08mm, symbol Coert-Vonk:TERM BLK PLG 2POS MSTB 5.08mm
- added PR5: LIGHT, symbol Coert-Vonk:PROBE_LIGHT
- D1: value SMBJ15A -> 15V
- P1, P2: now not fitted
- P4: value MAIN -> DC40-1250; UPC (none) -> 610395973836
- P7: value pH↓ -> NKP-DC-B08
- P8: value NUT_A -> NKP-DC-B08
- P9: value NUT_B -> NKP-DC-B08
- PR1: renamed from PB1; DKPN (none) -> 1528-2832-ND
- PR6: renamed from PB6; now not fitted
- V1: value ATO -> 2V025-08
- renumbered PB2 to PR2, PB3 to PR3, PB4 to PR4, DC1 to U2, U2 to U3, U3 to U4
Connections:
- net GND: now also H7.2
- net at P1.1: now also PR5.1
- net at P1.2: now also PR5.2
- net at P1.3: now also PR5.3
- net at P1.4: now also PR5.4
- net at F1.1: now also H7.1
- new net: DC1.12V, P10.1
- new net: DC1.GND, P10.2
Other:
- note removed: "12V DC Supply"
- moved on the sheet: C15, C20, C3, C4, C5, C6, C7, C8, D1, D6, F1, H5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
