File: hardware/OPNhydro_r2/OPNhydro_r2.kicad_sch (KiCad schematic)
At the start: 149 parts, among them J1 MKDS, J2 MKDS, J3 BNC, J4 BNC, J5 BNC, M1 ESP32-C6-DEVKIT, M2 pH, M3 EC, M4 RTD, P1 MSTB_0.2"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

Commit message: tweak layout
Other:
- note added: "MAIN PUMP & VALVE DRIVERS"
- note removed: "PUMP & VALVE DRIVERS"
- moved on the sheet: C10, C13, C14, C17, C18, C23, C24, C27, C28, C8, D2, D3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
